File: Hardware/CortexPC.kicad_pcb (KiCad board)
At the start: 2 copper layers, 244 x 244 mm, 131 parts, among them J1 F18A TANG NANO Connector, J10 Bus_I_not_SA_8bit, J11 IRQ Selection, J12 Bus_I_not_SA_8bit, J13 IRQ Selection, J14 Bus_I_not_SA_8bit, J15 IRQ Selection, J16 Bus_I_not_SA_8bit, J17 IRQ Selection, J18 Bus_I_not_SA_8bit, J19 Parallel Keyboard IN, J2 IRQ Selection, J3 Bus_I_not_SA_8bit, J4 Enable Serial Int, J5 TTL SERIAL 0, J6 TTL SER 0 PWR, J7 USER OUT, J8 IRQ Selection, J9 AUDIO OUT, P1 14.31818 MHz CLK, P10 CONN_1, P11 CONN_1, P12 CONN_1, P13 CONN_1, P14 CONN_1, P15 CONN_1, P16 CONN_1, P17 CONN_1, P18 CONN_1, P2 CONN_1, P4 8 BIT IDE (CF), P5 CONN_10X2, P6 POWER_SW, P7 CONN_1, P9 CONN_1, SW1 RESET, SW2 POWER, U1 74LS14, U10 TMS9918 EMU, U11 GAL22V10, U12 74LS32, U13 74LS32, U14 74LS244, U15 74LS138, U17 74LS688, U18 27C256, U2 74LS07, U21 TMS9902A, U22 74LS259, U23 74LS612-DIP, U25 74LS245, U26 74HCT14, U27 74LS74, U28 74LS244, U29 74LS244, U3 TMS9995-DIP_1, U30 GAL22V10, U31 74LS244, U4 74LS04, U5 74LS74, U6 74LS112, U7 SN76489, U8 DS1233, U9 SRAM_512K, Y1 12MHz

Commit message: Initial Commit
Routing:
- net GND: track 0.00 -> 2233.3 mm, vias 0 -> 2
- net VCC: track 0.00 -> 1643.7 mm
- net /RESET: track 0.00 -> 569.8 mm, vias 0 -> 1
- net +12V: track 0.00 -> 542.4 mm, vias 0 -> 8
- net -5V: track 0.00 -> 506.0 mm, vias 0 -> 3
- net CPU-D3: track 0.00 -> 497.0 mm, vias 0 -> 2
- net CPU-D2: track 0.00 -> 479.5 mm, vias 0 -> 2
- net CPU-D0: track 0.00 -> 456.1 mm, vias 0 -> 2
- net CPU-A0: track 0.00 -> 448.3 mm, vias 0 -> 2
- net CPU-D7: track 0.00 -> 436.8 mm, vias 0 -> 4
- net CPU-D5: track 0.00 -> 435.7 mm, vias 0 -> 2
- net CPU-D1: track 0.00 -> 434.5 mm, vias 0 -> 3
- net -12V: track 0.00 -> 429.8 mm, vias 0 -> 5
- net CPU-D6: track 0.00 -> 427.3 mm, vias 0 -> 3
- net CPU-D4: track 0.00 -> 421.9 mm, vias 0 -> 2
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- added copper zone on B.Cu, net GND
- added copper zone on F.Cu, net GND

Commit message: updates
Parts:
- removed U14: 74LS244, Custom:STD_DDW_DIP20
- added C36: 4.7pF, Custom:STD_DDW_CAP, F.Cu at (81.5, 205.7)
- added C37: 0.1 uF, Custom:STD_DDW_CAP, F.Cu at (57.5, 179.0)
- added C38: 0.22uf, Custom:STD_DDW_PCAP, F.Cu at (120.0, 177.7)
- added C39: 10uf, Custom:STD_DDW_PCAP, F.Cu at (113.6, 194.8)
- added C42: 2200pf, Custom:STD_DDW_CAP, F.Cu at (57.5, 185.6)
- added C43: 10uf, Custom:STD_DDW_PCAP, F.Cu at (113.6, 204.1)
- added C44: 470pf, Custom:STD_DDW_CAP, F.Cu at (57.5, 192.2)
- added C45: 470pf, Custom:STD_DDW_CAP, F.Cu at (57.5, 198.8)
- added C46: 2200pf, Custom:STD_DDW_CAP, F.Cu at (57.5, 205.3)
- added C47: 0.047uf, Custom:STD_DDW_CAP, F.Cu at (57.2, 211.9)
- added C48: 220uf, Custom:STD_DDW_PCAP, F.Cu at (113.7, 213.4)
- added C49: 10uf, Custom:STD_DDW_PCAP, F.Cu at (120.7, 194.6)
- added C50: 0.47uf, Custom:STD_DDW_PCAP, F.Cu at (121.2, 204.1)
- added C51: 1uf, Custom:STD_DDW_PCAP, F.Cu at (121.1, 213.8)
- added C53: 1uf, Custom:STD_DDW_PCAP, F.Cu at (94.5, 133.0)
- added C56: 0.047uf, Custom:STD_DDW_CAP, F.Cu at (81.4, 211.9)
- added C57: 220uf, Custom:STD_DDW_PCAP, F.Cu at (111.3, 133.1)
- added C58: 10uf, Custom:STD_DDW_PCAP, F.Cu at (102.8, 133.1)
- added J20: SID Speaker, Custom:STD_DDW_PINHEAD_V_1x02, F.Cu at (130.2, 165.2)
- added J21: SID AMP Enable, Custom:STD_DDW_PINHEAD_V_1x02, F.Cu at (118.8, 165.1)
- added J22: SN76489 AMP Enable, Custom:STD_DDW_PINHEAD_V_1x02, F.Cu at (57.1, 141.7)
- added J23: SN76489 Speaker, Custom:STD_DDW_PINHEAD_V_1x02, F.Cu at (57.1, 150.3)
- added J24: SID OUT, Custom:CUI_RCJ-047, F.Cu at (179.2, 21.2)
- added JP2: ENABLE KEYBOARD, Custom:STD_DDW_PINHEAD_V_1x02, F.Cu at (216.7, 79.5)
- added P3: 1 MHz CLK, Custom:STD_DDW_DIP14, F.Cu at (70.9, 148.1)
- added R15: 10 ohms, Custom:STD_DDW_RESISTOR, F.Cu at (44.7, 192.6)
- added R19: 4.3K, Custom:STD_DDW_RESISTOR, F.Cu at (44.5, 199.3)
- added R20: 22K, Custom:STD_DDW_RESISTOR, F.Cu at (44.5, 205.6)
- added R21: 470K, Custom:STD_DDW_RESISTOR, F.Cu at (44.5, 212.0)
- added R22: 470K, Custom:STD_DDW_RESISTOR, F.Cu at (68.7, 192.3)
- added R23: 22K, Custom:STD_DDW_RESISTOR, F.Cu at (68.6, 198.8)
- added R24: 10 ohms, Custom:STD_DDW_RESISTOR, F.Cu at (68.4, 205.9)
- added R25: 4.3K, Custom:STD_DDW_RESISTOR, F.Cu at (68.5, 212.3)
- added R26: 4.7K, Custom:STD_DDW_RESISTOR, F.Cu at (216.6, 64.5)
- added R27: 4.7K, Custom:STD_DDW_RESISTOR, F.Cu at (216.6, 70.8)
- added RV1: 1K, Potentiometer_THT:Potentiometer_Bourns_3386F_Vertical, F.Cu at (96.2, 189.8)
- added RV2: 1K, Potentiometer_THT:Potentiometer_Bourns_3386F_Vertical, F.Cu at (96.2, 202.7)
- added U16: 6581, Custom:STD_DDW_DIP28, F.Cu at (102.6, 157.1)
- added U19: 74LS374, Custom:STD_DDW_DIP20, F.Cu at (84.7, 151.9)
- added U20: 74LS374, Custom:STD_DDW_DIP20, F.Cu at (84.9, 183.3)
- added U24: LM386, Custom:STD_DDW_DIP8, F.Cu at (43.7, 161.5)
- added U32: LM386, Custom:STD_DDW_DIP8, F.Cu at (59.6, 161.6)
- added U33: ATtiny85-20P, Custom:STD_DDW_DIP8, F.Cu at (202.4, 52.8)
- J19: value Parallel Keyboard IN -> KEYBOARD; footprint Custom:STD_DDW_PinHeader_1x11 -> Custom:PS2_DIN
- moved J19 7.61 mm to (197.1, 25.2), turned to 0 degrees
Connections:
- J19 pad 1: VCC -> /IO/KBDDAT
- J19 pad 2: Net-(J19-Pin_2) -> unconnected-(J19-Pad2)
- J19 pad 3: Net-(J19-Pin_3) -> GND
- J19 pad 4: Net-(J19-Pin_4) -> VCC
- J19 pad 5: Net-(J19-Pin_5) -> /IO/KBDCLK
- J19 pad 6: Net-(J19-Pin_6) -> unconnected-(J19-Pad6)
- U11 pad 14: unconnected-(U11-O9-Pad14) -> ~{SIDSEL}
- U11 pad 16: ~{KeyboardSel} -> unconnected-(U11-O7-Pad16)
- U13 pad 11: unconnected-(U13-Pad11) -> Net-(U19-Cp)
- U13 pad 12: unconnected-(U13-Pad12) -> ~{SIDSEL}
- U13 pad 13: unconnected-(U13-Pad13) -> ~{PWE}
Routing:
- net GND: track 2233.3 -> 0.00 mm, vias 2 -> 0
- net VCC: track 1643.7 -> 0.00 mm
- net /RESET: track 569.8 -> 0.00 mm, vias 1 -> 0
- net +12V: track 542.4 -> 0.00 mm, vias 8 -> 0
- net -5V: track 506.0 -> 0.00 mm, vias 3 -> 0
- net CPU-D3: track 497.0 -> 0.00 mm, vias 2 -> 0
- net CPU-D2: track 479.5 -> 0.00 mm, vias 2 -> 0
- net CPU-D0: track 456.1 -> 0.00 mm, vias 2 -> 0
- net CPU-A0: track 448.3 -> 0.00 mm, vias 2 -> 0
- net CPU-D7: track 436.8 -> 0.00 mm, vias 4 -> 0
- net CPU-D5: track 435.7 -> 0.00 mm, vias 2 -> 0
- net CPU-D1: track 434.5 -> 0.00 mm, vias 3 -> 0
- net -12V: track 429.8 -> 0.00 mm, vias 5 -> 0
- net CPU-D6: track 427.3 -> 0.00 mm, vias 3 -> 0
- net CPU-D4: track 421.9 -> 0.00 mm, vias 2 -> 0
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- removed copper zone on B.Cu, net GND
- removed copper zone on F.Cu, net GND
Other:
- board text added: "CortexPC ATX rev. V0.50-000 6/14/2025 D. Werner https://github.com/danwerner21/CortexPC Licensed for hobbyist use only. All other rights reserved."
- board text removed: "CortexPC ATX rev. V0.50-000 5/25/2025 D. Werner https://github.com/danwerner21/CortexPC Licensed for hobbyist use only. All other rights reserved."

Commit message: notes
Routing:
- net GND: track 0.00 -> 2628.4 mm, vias 0 -> 1
- net VCC: track 0.00 -> 1884.8 mm, vias 0 -> 1
- net +12V: track 0.00 -> 667.8 mm, vias 0 -> 11
- net /RESET: track 0.00 -> 622.7 mm, vias 0 -> 2
- net CPU-A0: track 0.00 -> 596.0 mm, vias 0 -> 2
- net CPU-A1: track 0.00 -> 566.2 mm, vias 0 -> 3
- net CPU-D3: track 0.00 -> 525.2 mm, vias 0 -> 1
- net CPU-A2: track 0.00 -> 515.5 mm, vias 0 -> 4
- net CPU-A3: track 0.00 -> 490.8 mm, vias 0 -> 6
- net -12V: track 0.00 -> 489.9 mm, vias 0 -> 5
- net -5V: track 0.00 -> 488.1 mm, vias 0 -> 6
- net CPU-D0: track 0.00 -> 471.1 mm, vias 0 -> 6
- net CPU-D2: track 0.00 -> 462.1 mm, vias 0 -> 3
- net CPU-D7: track 0.00 -> 457.8 mm, vias 0 -> 5
- net CPU-D1: track 0.00 -> 444.0 mm, vias 0 -> 4
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- added copper zone on B.Cu, net GND
- added copper zone on F.Cu, net GND

Commit message: cortex work
Parts:
- removed C51, C53: 1uf, Custom:STD_DDW_PCAP
- removed R10: 10K, Custom:STD_DDW_RESISTOR
- removed R19, R25: 4.3K, Custom:STD_DDW_RESISTOR
- removed R20, R23: 22K, Custom:STD_DDW_RESISTOR
- removed R21, R22: 470K, Custom:STD_DDW_RESISTOR
- removed U1: 74LS14, Custom:STD_DDW_DIP14
- added JP3: SID CS, Custom:STD_DDW_PINHEAD_V_1x03, F.Cu at (85.1, 135.1)
- added R28: 10k, Custom:STD_DDW_RESISTOR, F.Cu at (121.9, 154.4)
- added R29: 10k, Custom:STD_DDW_RESISTOR, F.Cu at (122.1, 141.5)
- added R30: 10k, Custom:STD_DDW_RESISTOR, F.Cu at (121.9, 147.8)
- RV1, RV2: value 1K -> 10K
- moved C11 26.0 mm to (203.7, 105.2)
- moved U13 25.3 mm to (185.9, 112.4)
- moved U21 20.8 mm to (166.1, 114.6)
- moved C4 8.66 mm to (185.2, 96.2)
Connections:
- C49 pad 2: Net-(J20-Pin_2) -> Net-(C49-Pad2)
- C58 pad 2: Net-(J23-Pin_2) -> Net-(C58-Pad2)
- J10 pad 2: ~{RES_OUT} -> RESET
- J10 pad 20: BUSCLK -> CLK
- J12 pad 2: ~{RES_OUT} -> RESET
- J12 pad 20: BUSCLK -> CLK
- J14 pad 2: ~{RES_OUT} -> RESET
- J14 pad 20: BUSCLK -> CLK
- J16 pad 2: ~{RES_OUT} -> RESET
- J16 pad 20: BUSCLK -> CLK
- J18 pad 2: ~{RES_OUT} -> RESET
- J18 pad 20: BUSCLK -> CLK
- J24 pad 1: Net-(J21-Pin_1) -> GND
- J24 pad 2: GND -> Net-(J21-Pin_1)
- J3 pad 2: ~{RES_OUT} -> RESET
- J3 pad 20: BUSCLK -> CLK
- J9 pad 1: SNDOUT -> GND
- J9 pad 2: GND -> SNDOUT
- P4 pad 1: Net-(P4-Pin_1) -> RESET
- RV1 pad 2: Net-(C51-Pad1) -> Net-(J21-Pin_1)
- RV2 pad 2: Net-(C53-Pad1) -> Net-(J22-Pin_1)
- U12 pad 1: IOR -> unconnected-(U12-Pad1)
- U12 pad 11: SMEMW -> unconnected-(U12-Pad11)
- U12 pad 12: ~{CPU-MREQ} -> unconnected-(U12-Pad12)
- U12 pad 13: ~{PWE} -> unconnected-(U12-Pad13)
- U12 pad 2: SMEMR -> unconnected-(U12-Pad2)
- U12 pad 3: Net-(U1-Pad11) -> unconnected-(U12-Pad3)
- U13 pad 10: ~{DBIN} -> unconnected-(U13-Pad10)
- U13 pad 8: SMEMR -> unconnected-(U13-Pad8)
- U13 pad 9: ~{CPU-MREQ} -> unconnected-(U13-Pad9)
- U16 pad 8: GND -> SIDCS
- U24 pad 1: Net-(R19-Pad2) -> Net-(C49-Pad1)
- U24 pad 3: Net-(U24-+) -> Net-(J21-Pin_2)
- U24 pad 8: unconnected-(U24-GAIN-Pad8) -> Net-(C49-Pad2)
- U25 pad 1: Net-(U25-A->B) -> IOR
- U26 pad 14: VCC -> 5VSB
- U27 pad 14: VCC -> 5VSB
- U32 pad 1: Net-(R25-Pad2) -> Net-(C58-Pad1)
- U32 pad 3: Net-(U32-+) -> Net-(J22-Pin_2)
- U32 pad 8: unconnected-(U32-GAIN-Pad8) -> Net-(C58-Pad2)
- U4 pad 12: Net-(P4-Pin_1) -> RESET
- U7 pad 1: CPU-D2 -> CPU-D5
- U7 pad 10: CPU-D7 -> CPU-D0
- U7 pad 11: CPU-D6 -> CPU-D1
- U7 pad 12: CPU-D5 -> CPU-D2
- U7 pad 13: CPU-D4 -> CPU-D3
- U7 pad 15: CPU-D3 -> CPU-D4
- U7 pad 2: CPU-D1 -> CPU-D6
- U7 pad 3: CPU-D0 -> CPU-D7
- U7 pad 4: Net-(U7-READY) -> unconnected-(U7-READY-Pad4)
Routing:
- net RESET: track 0.00 -> 352.4 mm, vias 0 -> 4
- net CLK: track 168.5 -> 307.1 mm, vias 3 -> 1
- net ~{CPU-MREQ}: track 124.7 -> 0.00 mm, vias 1 -> 0
- net BUSCLK: track 311.8 -> 189.2 mm, vias 0 -> 3
- net Net-(U1-Pad11): track 117.5 -> 0.00 mm, vias 1 -> 0
- net Net-(P4-Pin_1): track 110.5 -> 0.00 mm, vias 1 -> 0
- net ~{RES_OUT}: track 107.9 -> 0.00 mm
- net -5V: track 488.1 -> 391.5 mm, vias 6 -> 2
- net VCC: track 1884.8 -> 1976.6 mm, vias 1 -> 6
- net Net-(C49-Pad2): track 0.00 -> 91.1 mm
- net B_INT: track 218.2 -> 301.9 mm, vias 3 -> 6
- net Net-(C53-Pad1): track 80.1 -> 0.00 mm
- net 5VSB: track 236.1 -> 309.5 mm, vias 1 -> 3
- net Net-(C58-Pad2): track 0.00 -> 69.7 mm, vias 0 -> 1
- net GND: track 2628.4 -> 2697.9 mm, vias 1 -> 4
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Other:
- board text added: "CortexPC ATX rev. V0.90-000 7/13/2025 D. Werner https://github.com/danwerner21/CortexPC Licensed for hobbyist use only. All other rights reserved."
- board text removed: "CortexPC ATX rev. V0.50-000 6/14/2025 D. Werner https://github.com/danwerner21/CortexPC Licensed for hobbyist use only. All other rights reserved."
