File: Hardware/CortexPC.kicad_sch (KiCad schematic)
At the start: 0 parts

Commit message: update with SID
Other:
- added sheet sid (sid.kicad_sch)
Changed lines of the file:
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@@
+	)
+	(sheet
+		(at 177.8 92.964)
+		(size 70.104 66.294)
+		(fields_autoplaced yes)
+		(stroke
+			(width 0.1524)
+			(type solid)
+		)
+		(fill
+			(color 0 0 0 0.0000)
+		)
+		(property "Sheetname" "sid"
+			(at 177.8 92.2524 0)
+			(effects
+				(font
+					(size 1.27 1.27)
+				)
+				(justify left bottom)
+			)
+		)
+		(property "Sheetfile" "sid.kicad_sch"
+			(at 177.8 159.8426 0)
+			(effects
+				(font
+					(size 1.27 1.27)
+				)
+				(justify left top)
+			)
+		)
+		(instances
+			(project "CortexPC"
+				(path "/18cdbc1e-88fb-4fa4-ad3d-e978304be174"
+					(page "9")
+				)
+			)
+		)
 	)
 	(sheet
