File: Hardware/GALS.kicad_sch (KiCad schematic)
At the start: 3 parts, among them U11 GAL22V10, U13 74LS32, U30 GAL22V10

Commit message: update with SID
Connections:
- net ~{SIDSEL}: now reaches U11.14 (O9)
- no-connect marks 10 -> 9
Other:
- note added: "The memory map is shown in the table below. Memory Address Mapped To >0000 - >7FFF ROM when enabled, otherwise RAM >8000 - >EFFF RAM >F000 - >F0FB TMS 9995 internal RAM >F0FC - >FDFF RAM >FE00 - >FE03 CF card ATA registers >FE10 - >FE13 SOUND >FE20 - >FE23 VIDEO >FE30 - >FE33 KEYBOARD >FE40 - >FE4F Memory mapper registers 0-15 >FE60 - >FE7F SID registers 0-31 >FE80 - >FEBF Offboard IO (ports $80-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"
- note removed: "The memory map is shown in the table below. Memory Address Mapped To >0000 - >7FFF ROM when enabled, otherwise RAM >8000 - >EFFF RAM >F000 - >F0FB TMS 9995 internal RAM >F0FC - >FDFF RAM >FE00 - >FE03 CF card ATA registers >FE10 - >FE13 SOUND >FE20 - >FE23 VIDEO >FE30 - >FE33 KEYBOARD >FE40 - >FE4F Memory mapper registers 0-15 >FE80 - >FEBF Offboard IO (ports $80-$FF) >FFF0 - >FFF9 RAM >FFFA - >F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"
Changed lines of the file:
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@@
-	)
-	(no_connect
-		(at 171.45 196.85)
 	)
 	(no_connect
@@
 		(pts
 			(xy 142.24 87.63) (xy 143.51 87.63)
+		)
+		(stroke
+			(width 0)
+			(type default)
+		)
+	)
+	(wire
+		(pts
+			(xy 171.45 196.85) (xy 173.99 196.85)
 		)
 		(stroke
@@
 		)
 	)
-	(text "The memory map is shown in the table below.\n\nMemory Address	Mapped To\n>0000 - >7FFF	ROM when enabled, otherwise RAM\n>8000 - >EFFF	RAM\n>F000 - >F0FB	TMS 9995 internal RAM\n>F0FC - >FDFF	RAM\n>FE00 - >FE03	CF card ATA registers \n>FE10 - >FE13	SOUND\n>FE20 - >FE23	VIDEO\n>FE30 - >FE33	KEYBOARD\n>FE40 - >FE4F	Memory mapper registers 0-15 \n>FE80 - >FEBF	Offboard IO (ports $80-$FF)\n>FFF0 - >FFF9	RAM\n>FFFA - >FFFF	TMS 9995 internal RAM\n\n\nCRU Address	Mapped To\n>0000 - >003F	TMS 9902 registers\n>0040 - >007F	Control signal latch (further details here)\n 	(Plus processor internal CRU bits)\n"
+	(text "The memory map is shown in the table below.\n\nMemory Address	Mapped To\n>0000 - >7FFF	ROM when enabled, otherwise RAM\n>8000 - >EFFF	RAM\n>F000 - >F0FB	TMS 9995 internal RAM\n>F0FC - >FDFF	RAM\n>FE00 - >FE03	CF card ATA registers \n>FE10 - >FE13	SOUND\n>FE20 - >FE23	VIDEO\n>FE30 - >FE33	KEYBOARD\n>FE40 - >FE4F	Memory mapper registers 0-15 \n>FE60 - >FE7F	SID registers 0-31 \n>FE80 - >FEBF	Offboard IO (ports $80-$FF)\n>FFF0 - >FFF9	RAM\n>FFFA - >FFFF	TMS 9995 internal RAM\n\n\nCRU Address	Mapped To\n>0000 - >003F	TMS 9902 registers\n>0040 - >007F	Control signal latch (further details here)\n 	(Plus processor internal CRU bits)\n"
 		(exclude_from_sim no)
 		(at 199.136 146.558 0)
@@
 		)
 	)
-	(text "=~{MEMEN}+~{ROMEN}+RA15\n=~{MEMEN}+~{ISFE}+!RA15+CPU-A7+CPU-A6+USER+CPU-A5+CPU-A4+~{CPU-A3}\n=~{MEMEN}+~{ISFE}+!RA15+CPU-A7+CPU-A6+USER+CPU-A5+CPU-A4+CPU-A3\n=~{MEMEN}+~{ISFE}+!RA15+CPU-A7+CPU-A6+USER+CPU-A5+CPU-A4\n=~{MEMEN}+~{ISFE}+!RA15+CPU-A7+CPU-A6+USER+CPU-A5+~{CPU-A4}+CPU-A3\n=!~{MEMEN}+~{ISFE}+RA15+CPU-A7+CPU-A6+USER\n=!~{ONBOARD_ROM}+!~{CFSEL}\n=~{MEMEN}+~{ISFE}+!RA15+CPU-A7+CPU-A6+USER+CPU-A5+~{CPU-A4}+~{CPU-A3}\n=~{MEMEN}+~{ISFE}+!~{CFSEL}+!~{MAPSEL}+!~{9902SEL}+USER+!RA15\n\n"
+	(text "=~{MEMEN}+~{ROMEN}+RA15\n=~{MEMEN}+~{ISFE}+!RA15+CPU-A7+CPU-A6+USER+CPU-A5+CPU-A4+~{CPU-A3}\n=~{MEMEN}+~{ISFE}+!RA15+CPU-A7+CPU-A6+USER+CPU-A5+CPU-A4+CPU-A3\n=~{MEMEN}+~{ISFE}+!RA15+CPU-A7+CPU-A6+USER+CPU-A5+CPU-A4\n=~{MEMEN}+~{ISFE}+!RA15+CPU-A7+CPU-A6+USER+CPU-A5+~{CPU-A4}+CPU-A3\n=!~{MEMEN}+~{ISFE}+RA15+CPU-A7+CPU-A6+USER\n=!~{ONBOARD_ROM}+!~{CFSEL}\n=~{MEMEN}+~{ISFE}+!RA15+CPU-A7+CPU-A6+USER+CPU-A5+~{CPU-A4}+~{CPU-A3}\n=~{MEMEN}+~{ISFE}+!~{CFSEL}+!~{MAPSEL}+!~{9902SEL}+USER+!RA15\n=~{MEMEN}+~{ISFE}+!RA15+CPU-A7+CPU-A6+USER+!CPU-A5\n"
 		(exclude_from_sim no)
 		(at 186.69 197.358 0)
@@
 			(effects
 				(font
+					(size 1.016 1.016)
+				)
+				(justify left)
+				(hide yes)
+			)
+		)
+	)
+	(global_label "~{SIDSEL}"
+		(shape output)
+		(at 173.99 196.85 0)
+		(fields_autoplaced yes)
+		(effects
+			(font
+				(size 1.016 1.016)
+			)
+			(justify left)
+		)
+		(property "Intersheetrefs" "${INTERSHEET_REFS}"
+			(at 181.0314 196.85 0)
+			(effects
+				(font

Commit message: updates
Connections:
- net ~{KeyboardSel}: no longer names the net of U11.16 (O7)
- no-connect marks 9 -> 10
Other:
- note added: "The memory map is shown in the table below. Memory Address Mapped To >0000 - >7FFF ROM when enabled, otherwise RAM >8000 - >EFFF RAM >F000 - >F0FB TMS 9995 internal RAM >F0FC - >FDFF RAM >FE00 - >FE03 CF card ATA registers >FE10 - >FE13 SOUND >FE20 - >FE23 VIDEO >FE40 - >FE4F Memory mapper registers 0-15 >FE60 - >FE7F SID registers 0-31 >FE80 - >FEBF Offboard IO (ports $80-$FF) >FFF0 - >FFF9 RAM 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"
- note removed: "The memory map is shown in the table below. Memory Address Mapped To >0000 - >7FFF ROM when enabled, otherwise RAM >8000 - >EFFF RAM >F000 - >F0FB TMS 9995 internal RAM >F0FC - >FDFF RAM >FE00 - >FE03 CF card ATA registers >FE10 - >FE13 SOUND >FE20 - >FE23 VIDEO >FE30 - >FE33 KEYBOARD >FE40 - >FE4F Memory mapper registers 0-15 >FE60 - >FE7F SID registers 0-31 >FE80 - >FEBF Offboard IO (ports $80-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"
Changed lines of the file:
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@@
+	)
+	(no_connect
+		(at 173.99 191.77)
 	)
 	(no_connect
@@
 		)
 	)
-	(text "The memory map is shown in the table below.\n\nMemory Address	Mapped To\n>0000 - >7FFF	ROM when enabled, otherwise RAM\n>8000 - >EFFF	RAM\n>F000 - >F0FB	TMS 9995 internal RAM\n>F0FC - >FDFF	RAM\n>FE00 - >FE03	CF card ATA registers \n>FE10 - >FE13	SOUND\n>FE20 - >FE23	VIDEO\n>FE30 - >FE33	KEYBOARD\n>FE40 - >FE4F	Memory mapper registers 0-15 \n>FE60 - >FE7F	SID registers 0-31 \n>FE80 - >FEBF	Offboard IO (ports $80-$FF)\n>FFF0 - >FFF9	RAM\n>FFFA - >FFFF	TMS 9995 internal RAM\n\n\nCRU Address	Mapped To\n>0000 - >003F	TMS 9902 registers\n>0040 - >007F	Control signal latch (further details here)\n 	(Plus processor internal CRU bits)\n"
+	(text "The memory map is shown in the table below.\n\nMemory Address	Mapped To\n>0000 - >7FFF	ROM when enabled, otherwise RAM\n>8000 - >EFFF	RAM\n>F000 - >F0FB	TMS 9995 internal RAM\n>F0FC - >FDFF	RAM\n>FE00 - >FE03	CF card ATA registers \n>FE10 - >FE13	SOUND\n>FE20 - >FE23	VIDEO\n>FE40 - >FE4F	Memory mapper registers 0-15 \n>FE60 - >FE7F	SID registers 0-31 \n>FE80 - >FEBF	Offboard IO (ports $80-$FF)\n>FFF0 - >FFF9	RAM\n>FFFA - >FFFF	TMS 9995 internal RAM\n\n\nCRU Address	Mapped To\n>0000 - >003F	TMS 9902 registers\n>0040 - >007F	Control signal latch (further details here)\n 	(Plus processor internal CRU bits)\n"
 		(exclude_from_sim no)
 		(at 199.136 146.558 0)
@@
 			(effects
 				(font
-					(size 1.27 1.27)
-				)
-				(justify left)
-				(hide yes)
-			)
-		)
-	)
-	(global_label "~{KeyboardSel}"
-		(shape output)
-		(at 173.99 191.77 0)
-		(fields_autoplaced yes)
-		(effects
-			(font
-				(size 1.016 1.016)
-			)
-			(justify left)
-		)
-		(property "Intersheetrefs" "${INTERSHEET_REFS}"
-			(at 185.1922 191.77 0)
-			(effects
-				(font

Commit message: cortex work
Connections:
- no-connect marks 10 -> 11
Other:
- note added: "The memory map is shown in the table below. Memory Address Mapped To >0000 - >7FFF ROM when enabled, otherwise RAM >8000 - >EFFF RAM >F000 - >F0FB TMS 9995 internal RAM >F0FC - >FDFF RAM >FE00 - >FE03 CF card ATA registers >FE08 - >FE08 SOUND >FE20 - >FE21 VIDEO >FE40 - >FE4F Memory mapper registers 0-15 >FE60 - >FE7F SID registers 0-31 >FE80 - >FEBF Offboard IO (ports $80-$FF) >FFF0 - >FFF9 RAM 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"
- note removed: "The memory map is shown in the table below. Memory Address Mapped To >0000 - >7FFF ROM when enabled, otherwise RAM >8000 - >EFFF RAM >F000 - >F0FB TMS 9995 internal RAM >F0FC - >FDFF RAM >FE00 - >FE03 CF card ATA registers >FE10 - >FE13 SOUND >FE20 - >FE23 VIDEO >FE40 - >FE4F Memory mapper registers 0-15 >FE60 - >FE7F SID registers 0-31 >FE80 - >FEBF Offboard IO (ports $80-$FF) >FFF0 - >FFF9 RAM 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"
Changed lines of the file:
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@@
 	(title_block
 		(title "CortexPC")
-		(date "2025-05-25")
-		(rev "V0.5")
+		(date "2025-07-13")
+		(rev "V0.9")
 	)
 	(no_connect
@@
 	(no_connect
 		(at 143.51 77.47)
+	)
+	(no_connect
+		(at 168.91 95.25)
 	)
 	(wire
@@
 		)
 	)
-	(text "The memory map is shown in the table below.\n\nMemory Address	Mapped To\n>0000 - >7FFF	ROM when enabled, otherwise RAM\n>8000 - >EFFF	RAM\n>F000 - >F0FB	TMS 9995 internal RAM\n>F0FC - >FDFF	RAM\n>FE00 - >FE03	CF card ATA registers \n>FE10 - >FE13	SOUND\n>FE20 - >FE23	VIDEO\n>FE40 - >FE4F	Memory mapper registers 0-15 \n>FE60 - >FE7F	SID registers 0-31 \n>FE80 - >FEBF	Offboard IO (ports $80-$FF)\n>FFF0 - >FFF9	RAM\n>FFFA - >FFFF	TMS 9995 internal RAM\n\n\nCRU Address	Mapped To\n>0000 - >003F	TMS 9902 registers\n>0040 - >007F	Control signal latch (further details here)\n 	(Plus processor internal CRU bits)\n"
+	(text "The memory map is shown in the table below.\n\nMemory Address	Mapped To\n>0000 - >7FFF	ROM when enabled, otherwise RAM\n>8000 - >EFFF	RAM\n>F000 - >F0FB	TMS 9995 internal RAM\n>F0FC - >FDFF	RAM\n>FE00 - >FE03	CF card ATA registers \n>FE08 - >FE08	SOUND\n>FE20 - >FE21	VIDEO\n>FE40 - >FE4F	Memory mapper registers 0-15 \n>FE60 - >FE7F	SID registers 0-31 \n>FE80 - >FEBF	Offboard IO (ports $80-$FF)\n>FFF0 - >FFF9	RAM\n>FFFA - >FFFF	TMS 9995 internal RAM\n\n\nCRU Address	Mapped To\n>0000 - >003F	TMS 9902 registers\n>0040 - >007F	Control signal latch (further details here)\n 	(Plus processor internal CRU bits)\n"
 		(exclude_from_sim no)
 		(at 199.136 146.558 0)
@@
 		(effects
 			(font
-				(size 1.016 1.016)
+				(size 1.15 1.15)
 			)
 			(justify right)
@@
 		(effects
 			(font
-				(size 1.016 1.016)
+				(size 1.15 1.15)
 			)
 			(justify right)
@@
 		(effects
 			(font
-				(size 1.016 1.016)
+				(size 1.15 1.15)
 			)
 			(justify right)
@@
 		(effects
 			(font
-				(size 1.016 1.016)
+				(size 1.15 1.15)
 			)
 			(justify right)
@@
 		(effects
 			(font
-				(size 1.016 1.016)
+				(size 1.15 1.15)
 			)
 			(justify right)
@@
 		(effects
 			(font
-				(size 1.016 1.016)
+				(size 1.15 1.15)
 			)
 			(justify right)
@@
 		(effects
 			(font
-				(size 1.016 1.016)
+				(size 1.15 1.15)
 			)
 			(justify left)
@@
 		(effects
 			(font
-				(size 1.016 1.016)
+				(size 1.15 1.15)
 			)
 			(justify right)
@@
 		(effects
 			(font
-				(size 1.016 1.016)
+				(size 1.15 1.15)
 			)
 			(justify right)
@@
 		(effects
 			(font
-				(size 1.016 1.016)
+				(size 1.15 1.15)
 			)
 			(justify right)
@@
 		(effects
 			(font
-				(size 1.016 1.016)
+				(size 1.15 1.15)
 			)
 			(justify right)
@@
 		(effects
 			(font
-				(size 1.016 1.016)
+				(size 1.15 1.15)
 			)
 			(justify right)
@@
 		(effects
 			(font
-				(size 1.016 1.016)
+				(size 1.15 1.15)
 			)
 			(justify left)
@@
 		(effects
 			(font
-				(size 1.016 1.016)
+				(size 1.15 1.15)
 			)
 			(justify left)
@@
 		(effects
 			(font
-				(size 1.016 1.016)
+				(size 1.15 1.15)
 			)
 			(justify right)
@@
 		(effects
 			(font
-				(size 1.016 1.016)
+				(size 1.15 1.15)
 			)
 			(justify right)
@@
 		(effects
 			(font
-				(size 1.016 1.016)
+				(size 1.15 1.15)
 			)
 			(justify left)
@@
 		(effects
 			(font
-				(size 1.27 1.27)
+				(size 1.15 1.15)
 			)
 			(justify left)
@@
 		(effects
 			(font
-				(size 1.016 1.016)
+				(size 1.15 1.15)
 			)
 			(justify right)
@@
 		(effects
 			(font
-				(size 1.016 1.016)
+				(size 1.15 1.15)
 			)
 			(justify right)
@@
 		(effects
 			(font
-				(size 1.27 1.27)
+				(size 1.15 1.15)
 			)
 			(justify left)
@@
 		(effects
 			(font
-				(size 1.016 1.016)
+				(size 1.15 1.15)
 			)
 			(justify right)
@@
 		(effects
 			(font
-				(size 1.016 1.016)
+				(size 1.15 1.15)
 			)
 			(justify right)
@@
 		(effects
 			(font
-				(size 1.016 1.016)
+				(size 1.15 1.15)
 			)
 			(justify left)
@@
 		(effects
 			(font
-				(size 1.016 1.016)
+				(size 1.15 1.15)
 			)
 			(justify left)
@@
 		(effects
 			(font
-				(size 1.016 1.016)
+				(size 1.15 1.15)
 			)
 			(justify right)
@@
 		(effects
 			(font
-				(size 1.016 1.016)
+				(size 1.15 1.15)
 			)
 			(justify left)
@@
 		(effects
 			(font
-				(size 1.016 1.016)
+				(size 1.15 1.15)
 			)
 			(justify left)
@@
 		(effects
 			(font
-				(size 1.016 1.016)
+				(size 1.15 1.15)
 			)
 			(justify right)
@@
 		(effects
 			(font
-				(size 1.016 1.016)
+				(size 1.15 1.15)
 			)
 			(justify right)
@@
 		(effects
 			(font
-				(size 1.27 1.27)
+				(size 1.15 1.15)
 			)
 			(justify left)
@@
 		(effects
 			(font
-				(size 1.016 1.016)
+				(size 1.15 1.15)
 			)
 			(justify right)
@@
 		(effects
 			(font
-				(size 1.016 1.016)
+				(size 1.15 1.15)
 			)
 			(justify left)
@@
 		(effects
 			(font
-				(size 1.016 1.016)
+				(size 1.15 1.15)
 			)
 			(justify left)
@@
 		(effects
 			(font
-				(size 1.016 1.016)
+				(size 1.15 1.15)
 			)
 			(justify right)
@@
 		(effects
 			(font
-				(size 1.016 1.016)
+				(size 1.15 1.15)
 			)
 			(justify right)
@@
 		(effects
 			(font
-				(size 1.016 1.016)
+				(size 1.15 1.15)
 			)
 			(justify left)
@@
 		(effects
 			(font
-				(size 1.016 1.016)
+				(size 1.15 1.15)
 			)
 			(justify left)
@@
 		(effects
 			(font
-				(size 1.016 1.016)
+				(size 1.15 1.15)
 			)
 			(justify right)
@@
 		(effects
 			(font
-				(size 1.016 1.016)
-			)
-			(justify right)
+				(size 1.15 1.15)
+			)
+			(justify right)
