File: Hardware/buffers.kicad_sch (KiCad schematic)
At the start: 11 parts, among them P1 14.31818 MHz CLK, U1 74LS14, U12 74LS32, U13 74LS32, U25 74LS245, U28 74LS244, U29 74LS244, U31 74LS244, U4 74LS04

Commit message: cortex work
Parts:
- removed U1: 74LS14, Custom:STD_DDW_DIP14, symbol 74xx:74LS14
- removed unit 4 of U12
- removed unit 1 of U12
- removed U13: 74LS32, Custom:STD_DDW_DIP14, symbol 74xx:74LS32
- added R29, R30: 10k, Custom:STD_DDW_RESISTOR, symbol Device:R
Connections:
- net GND: now also R29.1, R30.1
- net IOR: now also U25.1 (A->B)
- net SMEMR: now also R29.2
- net SMEMW: now also R30.2
