File: Hardware/bus.kicad_sch (KiCad schematic)
At the start: 12 parts, among them J10 Bus_I_not_SA_8bit, J11 IRQ Selection, J12 Bus_I_not_SA_8bit, J13 IRQ Selection, J14 Bus_I_not_SA_8bit, J15 IRQ Selection, J16 Bus_I_not_SA_8bit, J17 IRQ Selection, J18 Bus_I_not_SA_8bit, J2 IRQ Selection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

Commit message: cortex work
Parts:
- added R28: 10k, Custom:STD_DDW_RESISTOR, symbol Device:R
Connections:
- net BUSCLK: no longer J10.20 (CLK), J12.20 (CLK), J14.20 (CLK), J16.20 (CLK), J18.20 (CLK), J3.20 (CLK)
- net B_INT: now also R28.1
- net GND: now also R28.2
- net ~{RES_OUT} renamed RESET
- new net CLK: J10.20 (CLK), J12.20 (CLK), J14.20 (CLK), J16.20 (CLK), J18.20 (CLK), J3.20 (CLK)
