File: Hardware/io.kicad_sch (KiCad schematic)
At the start: 19 parts, among them J4 Enable Serial Int, J5 TTL SERIAL 0, J6 TTL SER 0 PWR, J7 USER OUT, P4 8 BIT IDE (CF), U2 74LS07, U21 TMS9902A, U22 74LS259, U4 74LS04

Commit message: updates
Parts:
- added J19: KEYBOARD, Custom:PS2_DIN, symbol Connector:Mini-DIN-6
- added JP2: ENABLE KEYBOARD, Custom:STD_DDW_PINHEAD_V_1x02, symbol Connector_Generic:Conn_01x02
- added R26, R27: 4.7K, Custom:STD_DDW_RESISTOR, symbol Device:R
- added U33: ATtiny85-20P, Custom:STD_DDW_DIP8, symbol MCU_Microchip_ATtiny:ATtiny85-20P
Connections:
- net GND: now also J19.3, U33.4 (GND)
- net RX: now also JP2.1 (Pin_1)
- net VCC: now also J19.4, R26.1, R27.1, U33.8 (VCC)
- new net: JP2.2 (Pin_2), U33.5 (AREF/PB0)
- new net KBDCLK: J19.5, R26.2, U33.7 (PB2)
- new net KBDDAT: J19.1, R27.2, U33.6 (PB1)
- no-connect marks 16 -> 18

Commit message: cortex work
Connections:
- net RESET: now reaches P4.1 (Pin_1), U4.12
- no-connect marks 18 -> 21
