File: Hardware/power.kicad_sch (KiCad schematic)
At the start: 62 parts, among them P10 CONN_1, P11 CONN_1, P12 CONN_1, P13 CONN_1, P14 CONN_1, P15 CONN_1, P16 CONN_1, P17 CONN_1, P18 CONN_1, P2 CONN_1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

Commit message: update with SID
Parts:
- removed unit 4 of U13
Connections:
- no-connect marks 31 -> 28
Changed lines of the file:
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@@
 	)
 	(no_connect
-		(at 36.83 71.12)
-	)
-	(no_connect
 		(at 48.26 63.5)
 	)
@@
 	)
 	(no_connect
-		(at 21.59 68.58)
-	)
-	(no_connect
 		(at 48.26 54.61)
 	)
@@
 		(at 21.59 83.82)
 	)
-	(no_connect
-		(at 21.59 73.66)
-	)
 	(wire
 		(pts
@@
 				)
 			)
-		)
-	)
-	(symbol
-		(lib_id "74xx:74LS32")
-		(at 29.21 71.12 0)
-		(unit 4)
-		(exclude_from_sim no)
-		(in_bom yes)
-		(on_board yes)
-		(dnp no)
-		(fields_autoplaced yes)
-		(property "Reference" "U13"
-			(at 29.21 62.23 0)
-			(effects
-				(font
-					(size 1.27 1.27)
-				)
-			)
-		)
-		(property "Value" "74LS32"
-			(at 29.21 64.77 0)
-			(effects
-				(font
-					(size 1.27 1.27)
-				)
-			)
-		)
-		(property "Footprint" "Custom:STD_DDW_DIP14"
-			(at 29.21 71.12 0)
-			(effects
-				(font
-					(size 1.27 1.27)
-				)
-				(hide yes)
-			)
-		)
-		(property "Datasheet" "http://www.ti.com/lit/gpn/sn74LS32"
-			(at 29.21 71.12 0)
-			(effects
-				(font
-					(size 1.27 1.27)
-				)
-				(hide yes)
-			)
-		)
-		(property "Description" "Quad 2-input OR"
-			(at 29.21 71.12 0)
-			(effects
-				(font
-					(size 1.27 1.27)
-				)
-				(hide yes)
-			)
-		)
-		(pin "7"
-		)
-		(pin "11"
-		)
-		(pin "6"
-		)
-		(pin "14"
-		)
-		(pin "9"
-		)
-		(pin "4"
-		)
-		(pin "13"
-		)
-		(pin "5"
-		)
-		(pin "2"
-		)
-		(pin "8"
-		)
-		(pin "1"
-		)
-		(pin "12"
-		)
-		(pin "10"
-		)
-		(pin "3"
-		)
-		(instances
-			(project "CortexPC"
-				(path "/18cdbc1e-88fb-4fa4-ad3d-e978304be174/00000000-0000-0000-0000-0000643138dc"
-					(reference "U13")
-					(unit 4)
-				)
-			)

Commit message: cortex work
Parts:
- removed U1: 74LS14, Custom:STD_DDW_DIP14, symbol 74xx:74LS14
- added unit 4 of U12
- added unit 1 of U12
- added unit 3 of U13
Connections:
- net 5VSB: now also U26.14 (VCC), U27.14 (VCC)
- net VCC: no longer U26.14 (VCC), U27.14 (VCC)
- no-connect marks 28 -> 27
Other:
- moved on the sheet: U26G, U27B, U27C
