File: Hardware/sid.kicad_sch (KiCad schematic)
At the start: 27 parts, among them J20 SID Speaker, J21 SID AMP Enable, J24 SID OUT, P3 1 MHz CLK, U13 74LS32, U16 6581, U19 74LS374, U20 74LS374, U24 LM386

Commit message: updates
Parts:
- RV1: footprint Custom:STD_DDW_RESISTOR -> Potentiometer_THT:Potentiometer_Bourns_3386F_Vertical
Changed lines of the file:
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@@
 			)
 		)
-		(property "Footprint" "Custom:STD_DDW_RESISTOR"
+		(property "Footprint" "Potentiometer_THT:Potentiometer_Bourns_3386F_Vertical"
 			(at 138.43 62.23 0)
 			(effects

Commit message: cortex work
Parts:
- removed C51: 1uf, Custom:STD_DDW_PCAP, symbol Device:C_Polarized_Small
- removed R19: 4.3K, Custom:STD_DDW_RESISTOR, symbol Device:R_Small
- removed R20: 22K, Custom:STD_DDW_RESISTOR, symbol Device:R_Small
- removed R21: 470K, Custom:STD_DDW_RESISTOR, symbol Device:R_Small
- added JP3: SID CS, Custom:STD_DDW_PINHEAD_V_1x03, symbol Connector_Generic:Conn_01x03
- RV1: value 1K -> 10K
Connections:
- net GND: now also J24.1 (In), JP3.1 (Pin_1); no longer J24.2 (Ext), U16.8 (~{CS})
- net SIDCLK: now also JP3.3 (Pin_3)
- net at RV1.2: now also J21.1 (Pin_1), J24.2 (Ext)
- net at J21.2 (Pin_2): now also U24.3 (+)
- net at C48.2, J20.2 (Pin_2): no longer C49.2
- net at C49.1: now also U24.1 (GAIN)
- net at U24.8 (GAIN): now also C49.2
- new net SIDCS: JP3.2 (Pin_2), U16.8 (~{CS})
- no-connect marks 13 -> 12
Other:
- note added: "* This looks wrong, but is correct on the footprint"
- note added: "Some SID replacement chips ignore the clock signal and requre CS to function properly. Set this jumper if your SID chip does not function."
- moved on the sheet: C49, J24
