File: Hardware/video.kicad_sch (KiCad schematic)
At the start: 11 parts, among them J1 F18A TANG NANO Connector, J19 Parallel Keyboard IN, J9 AUDIO OUT, U10 TMS9918 EMU, U14 74LS244, U7 SN76489

Commit message: update with SID
Parts:
- added C36: 4.7pF, Custom:STD_DDW_CAP, symbol Device:C
- added C53: 1uf, Custom:STD_DDW_PCAP, symbol Device:C_Polarized_Small
- added C56: 0.047uf, Custom:STD_DDW_CAP, symbol Device:C_Small
- added C57: 220uf, Custom:STD_DDW_PCAP, symbol Device:C_Polarized_Small
- added C58: 10uf, Custom:STD_DDW_PCAP, symbol Device:C_Polarized_Small
- added J22: SN76489 AMP Enable, Custom:STD_DDW_PINHEAD_V_1x02, symbol Connector:Conn_01x02_Pin
- added J23: SN76489 Speaker, Custom:STD_DDW_PINHEAD_V_1x02, symbol Connector:Conn_01x02_Pin
- added R22: 470K, Custom:STD_DDW_RESISTOR, symbol Device:R_Small
- added R23: 22K, Custom:STD_DDW_RESISTOR, symbol Device:R_Small
- added R24: 10 ohms, Custom:STD_DDW_RESISTOR, symbol Device:R_Small
- added R25: 4.3K, Custom:STD_DDW_RESISTOR, symbol Device:R_Small
- added RV2: 1K, Custom:STD_DDW_RESISTOR, symbol Device:R_Potentiometer_Small
- added U32: LM386, Custom:STD_DDW_DIP8, symbol Amplifier_Audio:LM386
Connections:
- net CPU-A0: now also C36.1
- net GND: now also C36.2, J23.1 (Pin_1), R23.2, R24.2, RV2.3, U32.2 (-), U32.4 (GND)
- net SNDOUT: now also RV2.1
- new net: C58.1, R25.1
- new net: C57.2, C58.2, J23.2 (Pin_2)
- new net: C56.1, C57.1, U32.5
- new net: C56.2, R24.1
- new net: J22.2 (Pin_2), R22.1
- new net: R22.2, R23.1, U32.3 (+)
- new net: R25.2, U32.1 (GAIN)
- new net: C53.2, J22.1 (Pin_1)
- new net: C53.1, RV2.2
- new net +12V: U32.6 (V+)
- no-connect marks 30 -> 32
Other:
- note added: "Next version needs a keyboard strobe (interrupt?). A VT82C42 keyboard controller would probably be best."
- note added: "Note that the sound chip relies on the Video chip/emulator to generate clock. Sound will not function without video present."

Commit message: updates
Parts:
- removed J19: Parallel Keyboard IN, Custom:STD_DDW_PinHeader_1x11, symbol Connector:Conn_01x11_Pin
- removed U14: 74LS244, Custom:STD_DDW_DIP20, symbol 74xx:74LS244
- RV2: footprint Custom:STD_DDW_RESISTOR -> Potentiometer_THT:Potentiometer_Bourns_3386F_Vertical
Other:
- note removed: "Next version needs a keyboard strobe (interrupt?). A VT82C42 keyboard controller would probably be best."

Commit message: cortex work
Parts:
- removed C53: 1uf, Custom:STD_DDW_PCAP, symbol Device:C_Polarized_Small
- removed R10: 10K, Custom:STD_DDW_RESISTOR, symbol Device:R
- removed R22: 470K, Custom:STD_DDW_RESISTOR, symbol Device:R_Small
- removed R23: 22K, Custom:STD_DDW_RESISTOR, symbol Device:R_Small
- removed R25: 4.3K, Custom:STD_DDW_RESISTOR, symbol Device:R_Small
- RV2: value 1K -> 10K
Connections:
- net CPU-D0: now also U7.10 (D7); no longer U7.3 (D0)
- net CPU-D1: now also U7.11 (D6); no longer U7.2 (D1)
- net CPU-D2: now also U7.12 (D5); no longer U7.1 (D2)
- net CPU-D3: now also U7.13 (D4); no longer U7.15 (D3)
- net CPU-D4: now also U7.15 (D3); no longer U7.13 (D4)
- net CPU-D5: now also U7.1 (D2); no longer U7.12 (D5)
- net CPU-D6: now also U7.2 (D1); no longer U7.11 (D6)
- net CPU-D7: now also U7.3 (D0); no longer U7.10 (D7)
- net GND: now also J9.1 (In); no longer J9.2 (Ext)
- net SNDOUT: now also J9.2 (Ext); no longer J9.1 (In)
- net at C58.1: now also U32.1 (GAIN)
- net at C57.2, J23.2 (Pin_2): no longer C58.2
- net at J22.2 (Pin_2): now also U32.3 (+)
- net at U32.8 (GAIN): now also C58.2
- net at J22.1 (Pin_1): now also RV2.2
Other:
- note added: "* This looks wrong, but is correct on the footprint"
- moved on the sheet: C58, J9
